Commit message: feat: update params for joint and axis and position

File: ic_arm_urdf/urdf/ic1.1.2.urdf (robot description, URDF)
Before this commit: robot ic1.1.2, 6 links, 5 joints
Links:
- link base_link: geometry collision mesh filename=/Users/lr-2002/project/instantcreation/IC_arm_control/ic_ar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; visual mesh filename=/Users/lr-2002/project/instantcreation/IC_arm_control/ic_ar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
- link l1: geometry collision mesh filename=/Users/lr-2002/project/instantcreation/IC_arm_control/ic_ar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; visual mesh filename=/Users/lr-2002/project/instantcreation/IC_arm_control/ic_ar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
- link l2: geometry collision mesh filename=/Users/lr-2002/project/instantcreation/IC_arm_control/ic_ar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; visual mesh filename=/Users/lr-2002/project/instantcreation/IC_arm_control/ic_ar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
- link l3: geometry collision mesh filename=/Users/lr-2002/project/instantcreation/IC_arm_control/ic_ar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; visual mesh filename=/Users/lr-2002/project/instantcreation/IC_arm_control/ic_ar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
- link l4: geometry collision mesh filename=/Users/lr-2002/project/instantcreation/IC_arm_control/ic_ar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; visual mesh filename=/Users/lr-2002/project/instantcreation/IC_arm_control/ic_ar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
- link l5: geometry collision mesh filename=/Users/lr-2002/project/instantcreation/IC_arm_control/ic_ar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; visual mesh filename=/Users/lr-2002/project/instantcreation/IC_arm_control/ic_ar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
Joints:
- joint j1: type continuous -> revolute
- joint j2: origin xyz=0.176971378800704 -0.0552999999999993 0 rpy=0 0.928321523209396 -1.57079632679489 -> xyz=0.176971378800704 -0.0552999999999993 0 rpy=0 1.57 -1.57079632679489
- joint j3: axis 1 0 0 -> -1 0 0; origin xyz=0.239291817338248 0.0267286211992953 0 rpy=-1.5210959256661 0 3.14159265358979 -> xyz=0.239291817338248 0.0267286211992953 0 rpy=-1.2 0 3.14
- joint j4: axis 0 1 0 -> 0 -1 0; origin xyz=-0.129008182661752 0 0 rpy=0 0.0539834371308359 0 -> xyz=-0.129008182661752 0 0 rpy=0 2.5 0

Commit message: feat: update urdf

File: ic_arm_urdf/urdf/ic1.1.2.urdf (robot description, URDF)
Before this commit: robot ic1.1.2, 6 links, 5 joints
Joints:
- joint j3: origin xyz=0.239291817338248 0.0267286211992953 0 rpy=-1.2 0 3.14 -> xyz=0.239291817338248 0.0267286211992953 0 rpy=-0 0 3.14
- joint j4: origin xyz=-0.129008182661752 0 0 rpy=0 2.5 0 -> xyz=-0.129008182661752 0 0 rpy=0 0 0

Commit message: feat: related part

File: ic_arm_urdf/urdf/ic1.1.2.urdf (robot description, URDF)
Before this commit: robot ic1.1.2, 6 links, 5 joints
Links:
- added link base_root_marker, mass 0.001; collision sphere radius=0.01; visual sphere radius=0.01
Joints:
- added joint base_to_marker: type fixed, parent base_root_marker, child base_link, origin xyz=0.47073 0.121 -0.2423 rpy=1.57 0 0
- joint j1: origin xyz=-0.29856 0.0020693 0.21104 rpy=1.5708 0 1.1547 -> xyz=-0.29856 0.0020693 0.21104 rpy=1.5708 0. 1.4647; type revolute -> continuous
- joint j4: origin xyz=-0.129008182661752 0 0 rpy=0 0 0 -> xyz=-0.129008182661752 0 0 rpy=0 0.087 0
- joint j5: axis 0 0 1 -> 0 0 -1

Commit message: feat: update urdf pos

File: ic_arm_urdf/urdf/ic1.1.2.urdf (robot description, URDF)
Before this commit: robot ic1.1.2, 7 links, 6 joints
Joints:
- joint j1: origin xyz=-0.29856 0.0020693 0.21104 rpy=1.5708 0. 1.4647 -> xyz=-0.29856 0.0020693 0.21104 rpy=1.5708 0. 1.6047
