Commit message: feat: sync new arm with 6248

File: ic_arm/urdf/ic_arm_rev.urdf (robot description, URDF)
Before this commit: robot ic_arm, 12 links, 11 joints
Joints:
- joint m1-l2: type continuous -> revolute
- joint m2-l3: type continuous -> revolute
- joint m3-l4: type continuous -> revolute
- joint m4-l5: type continuous -> revolute
- joint m5-l6: type continuous -> revolute
