Commit message: feat: update axis

File: robot/urdf/robot.urdf (robot description, URDF)
Before this commit: robot robot, 6 links, 5 joints
Joints:
- joint joint3: axis 0 0 -1 -> 0 0 1

Commit message: feat: gravity compensation tested : init version

File: robot/urdf/robot.urdf (robot description, URDF)
Before this commit: robot robot, 6 links, 5 joints
Links:
- link base_link: geometry collision mesh filename=/Users/lr-2002/project/instantcreation/IC_arm_control/robot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; visual mesh filename=/Users/lr-2002/project/instantcreation/IC_arm_control/robot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
- link joint1_link: geometry collision mesh filename=/Users/lr-2002/project/instantcreation/IC_arm_control/robot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; visual mesh filename=/Users/lr-2002/project/instantcreation/IC_arm_control/robot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
- link joint2_link: geometry collision mesh filename=/Users/lr-2002/project/instantcreation/IC_arm_control/robot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; visual mesh filename=/Users/lr-2002/project/instantcreation/IC_arm_control/robot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
- link joint3_link: geometry collision mesh filename=/Users/lr-2002/project/instantcreation/IC_arm_control/robot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; visual mesh filename=/Users/lr-2002/project/instantcreation/IC_arm_control/robot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
- link joint4_link: geometry collision mesh filename=/Users/lr-2002/project/instantcreation/IC_arm_control/robot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; visual mesh filename=/Users/lr-2002/project/instantcreation/IC_arm_control/robot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
- link joint5_link: geometry collision mesh filename=/Users/lr-2002/project/instantcreation/IC_arm_control/robot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; visual mesh filename=/Users/lr-2002/project/instantcreation/IC_arm_control/robot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
