Commit message: feat: updated urdf

File: robot_8dof/urdf/robot_8dof_updated.urdf (robot description, URDF)
Before this commit: robot robot_8dof, 7 links, 6 joints
Joints:
- joint joint2: limit lower=-0.184733 upper=3.468856 effort=100.0 velocity=3.14 -> lower=-0.184733 upper=3.468856 effort=27 velocity=3.14
- joint joint3: limit lower=-0.651685 upper=3.486621 effort=100.0 velocity=3.14 -> lower=-0.651685 upper=3.486621 effort=60 velocity=3.14
- joint joint4: limit lower=-3.464279 upper=1.971183 effort=100.0 velocity=3.14 -> lower=-3.464279 upper=1.971183 effort=27 velocity=3.14
- joint joint5: limit lower=-1.694232 upper=1.804860 effort=100.0 velocity=3.14 -> lower=-1.694232 upper=1.804860 effort=27 velocity=3.14
- joint joint6: limit lower=-2.072274 upper=4.018944 effort=100.0 velocity=3.14 -> lower=-2.072274 upper=4.018944 effort=27.0 velocity=3.14
