Commit message: feat: update urdf axis

File: urdfs/ic_arm_8_dof/urdf/ic_arm_8_dof.urdf (robot description, URDF)
Before this commit: robot ic_arm_8_dof, 7 links, 6 joints
Joints:
- joint joint1: axis 0 0 -1 -> 0 0 1
- joint joint2: axis 0 0 -1 -> 0 0 1
- joint joint3: axis 0 0 -1 -> 0 0 1
- joint joint4: axis 0 0 -1 -> 0 0 1

Commit message: feat: update urdf limit

File: urdfs/ic_arm_8_dof/urdf/ic_arm_8_dof.urdf (robot description, URDF)
Before this commit: robot ic_arm_8_dof, 7 links, 6 joints
Joints:
- joint joint1: limit lower=-3.14 upper=3.14 effort=0 velocity=0 -> lower=-1.383330 upper=0.300702 effort=100.0 velocity=3.14
- joint joint2: limit lower=-3.14 upper=3.14 effort=0 velocity=0 -> lower=-3.063722 upper=0.433749 effort=100.0 velocity=3.14
- joint joint3: limit lower=-3.14 upper=3.14 effort=0 velocity=0 -> lower=-0.484754 upper=2.041338 effort=100.0 velocity=3.14
- joint joint4: limit lower=-3.14 upper=3.14 effort=0 velocity=0 -> lower=-3.006890 upper=2.259960 effort=100.0 velocity=3.14
- joint joint5: limit lower=-3.14 upper=3.14 effort=0 velocity=0 -> lower=-1.769764 upper=1.739628 effort=100.0 velocity=3.14
- joint joint6: limit lower=-3.14 upper=3.14 effort=0 velocity=0 -> lower=-2.071130 upper=3.858724 effort=100.0 velocity=3.14

Commit message: feat: update ic_arm urdf

File: urdfs/ic_arm_8_dof/urdf/ic_arm_8_dof.urdf (robot description, URDF)
Before this commit: robot ic_arm_8_dof, 7 links, 6 joints
Joints:
- joint joint1: limit lower=-1.383330 upper=0.300702 effort=100.0 velocity=3.14 -> lower=-1.383330 upper=0.300702 effort=130 velocity=1.57
- joint joint2: limit lower=-3.063722 upper=0.433749 effort=100.0 velocity=3.14 -> lower=-3.063722 upper=0.433749 effort=80.0 velocity=1.57
- joint joint3: limit lower=-0.484754 upper=2.041338 effort=100.0 velocity=3.14 -> lower=-0.484754 upper=2.041338 effort=80.0 velocity=1.57
- joint joint4: limit lower=-3.006890 upper=2.259960 effort=100.0 velocity=3.14 -> lower=-3.006890 upper=2.259960 effort=27 velocity=1.57
- joint joint5: limit lower=-1.769764 upper=1.739628 effort=100.0 velocity=3.14 -> lower=-1.769764 upper=1.739628 effort=27. velocity=1.57
- joint joint6: limit lower=-2.071130 upper=3.858724 effort=100.0 velocity=3.14 -> lower=-2.071130 upper=3.858724 effort=10.0 velocity=1.57
