Commit message: feat: urdfs

File: urdfs/ic_arm_8_dof/urdf/ic_arm_8_dof_last_updated.urdf (robot description, URDF)
Before this commit: robot ic_arm_8_dof, 7 links, 6 joints
Joints:
- joint joint1: limit lower=-0.326261 upper=0.560105 effort=100.0 velocity=3.14 -> lower=-1.210903 upper=0.096994 effort=100.0 velocity=3.14
- joint joint2: limit lower=-1.982664 upper=0.556083 effort=100.0 velocity=3.14 -> lower=-2.157152 upper=0.546879 effort=100.0 velocity=3.14
- joint joint3: limit lower=-0.467113 upper=0.664994 effort=100.0 velocity=3.14 -> lower=-0.460210 upper=2.045557 effort=100.0 velocity=3.14
- joint joint4: limit lower=-0.503647 upper=3.236919 effort=100.0 velocity=3.14 -> lower=-3.007653 upper=1.863989 effort=100.0 velocity=3.14
- joint joint5: limit lower=-0.629915 upper=1.244091 effort=100.0 velocity=3.14 -> lower=-1.707965 upper=1.849874 effort=100.0 velocity=3.14
- joint joint6: limit lower=-1.237606 upper=1.555757 effort=100.0 velocity=3.14 -> lower=-1.374174 upper=3.468094 effort=100.0 velocity=3.14
